Commit message: lab4

File: src/my_r2d2/urdf/r2d2.xacro (robot description, xacro)
@@ -232,3 +232,11 @@
     <origin rpy="0 ${pi/2} 0" xyz="0 0 0"/>
   </joint>
+    <link name="base_footprint">
+    </link>
+    <joint name="from_base_footprint" type="fixed">
+      <axis xyz="0 1 0" rpy="0 0 0" />
+      <parent link="base_footprint"/>
+      <child link="base_link"/>
+      <origin xyz="0 0 ${(bodylen/2)+0.1+wheeldiam}" rpy="0 0 0"/>
+    </joint>
 </robot>

Commit message: camera

File: src/my_r2d2/urdf/r2d2.xacro (robot description, xacro)
@@ -219,4 +219,5 @@
       </geometry>
       <material name="black"/>
+	<origin rpy="0 ${pi/2} 0" xyz="0 0 0"/>
     </visual>
     <collision>
@@ -230,5 +231,5 @@
     <parent link="box"/>
     <child link="lens"/>
-    <origin rpy="0 ${pi/2} 0" xyz="0 0 0"/>
+    <origin rpy="0 0 0" xyz="0 0 0"/>
   </joint>
     <link name="base_footprint">
@@ -240,3 +241,10 @@
       <origin xyz="0 0 ${(bodylen/2)+0.1+wheeldiam}" rpy="0 0 0"/>
     </joint>
+  <link name="eye">
+  </link>
+  <joint name="camlens" type="continuous">
+    <parent link="lens"/>
+    <child link="eye"/>
+    <origin rpy="${pi/2} ${pi} ${pi/2}" xyz="0 0 0"/>
+  </joint>
 </robot>
