Commit message: update

File: src/my_r2d2/urdf/r2d2.urdf (robot description, URDF)
Before this commit: robot physics, 16 links, 15 joints
Links:
- link base_link: mass 10 -> None
- link right_leg: mass 10 -> None

File: src/my_r2d2/urdf/r2d2.xacro (robot description, xacro)
@@ -216,20 +216,18 @@
     <visual>
       <geometry>
-        <cylinder length="0.01" radius="0.03"/>
+        <cylinder radius="0.03" length="0.02"/>
       </geometry>
       <material name="black"/>
-	<origin rpy="0 ${pi/2} 0" xyz="0 0 0"/>
-    </visual>
-    <collision>
-      <geometry>
-        <cylinder length="0.01" radius="0.03"/>
-      </geometry>
-    </collision>
-    <xacro:default_inertial mass="1"/>
+    </visual>
+    <collision>
+      <geometry>
+        <cylinder radius="0.03" length="0.02"/>
+      </geometry>
+    </collision>
   </link>
   <joint name="tolens" type="fixed">
     <parent link="box"/>
     <child link="lens"/>
-    <origin rpy="0 0 0" xyz="0 0 0"/>
+    <origin rpy="0 ${pi/2} 0" xyz="0.01 0 0"/>
   </joint>
     <link name="base_footprint">
